Commit message: Just a leg

File: WalkingSimulation/Leg.urdf (robot description, URDF)
Before this commit: robot Stomp, 6 links, 5 joints
Links:
- removed link pivot_cylinder
- removed link pivot_rod
Joints:
- removed joint pivot_cylinder_base
- removed joint pivot_cylinder_slide
- joint pivot: origin xyz=0.0 0.0 0.112 rpy=0 0 0 -> xyz=0.0 -0.11 0.11 rpy=0 0 0
